File: _autosave-KicadJE_uP_DAC.kicad_pcb (KiCad board)
At the start: 2 copper layers, 100 x 100 mm, 216 parts, among them J201 CV1, J202 CV2, J203 OUT1, J204 OUT2, J205 IN1, J206 IN2, J301 AVR-ISP-6, J302 UART, J401 CV1, J402 CV2, J403 OUT1, J404 OUT2, J405 OUT3, J406 OUT4, J407 IN1, J408 IN2, J409 I2C, J501 BOOT, J502 UART, J503 USB_B_Micro, P201 Doepfer_Power_16pin, P401 Doepfer_Power_16pin, SW201 SW_SPDT, SW401 SW_SPDT, U201 TL072, U202 MCP4822, U301 ATmega32A-AU, U401 TL072, U402 TL072, U405 MCP4822, U501 AMS1117-3.3, U502 STM32F103C8Tx, Y301 16MHz, Y501 8 MHz

Commit message: Diode etc
Parts:
- removed D402, D403, D405, D406, D407, D410, D411, D412, D415, D416, D417: LED, LED_THT:LED_D3.0mm
- removed R429, R430, R431, R432, R433, R434: 100R, Resistor_SMD:R_0805_2012Metric_Pad1.15x1.40mm_HandSolder
- R437: value 100R -> 820R; moved to F.Cu
- moved D401 86.4 mm to (84.0, 106.0), turned to 270 degrees
- moved R437 43.9 mm to (81.0, 107.0), turned to 180 degrees
Connections:
- D401 pad 1: PB4_C0 -> GND
- D401 pad 2: PB0_R0 -> Net-(D401-Pad2)
- JP407 pad 2: /KicadJE_STM32F0/STM32F103C8/STM32_SDA1_PWM_PB9 -> PB9_PWM
- R437 pad 1: (no net) -> Net-(D401-Pad2)
- R437 pad 2: PA15_C2 -> PB9_PWM
- R506 pad 2: /KicadJE_STM32F0/STM32F103C8/STM32_boot1_PB2 -> PB2_R2
- U502 pad 20: /KicadJE_STM32F0/STM32F103C8/STM32_boot1_PB2 -> PB2_R2
- U502 pad 46: /KicadJE_STM32F0/STM32F103C8/STM32_SDA1_PWM_PB9 -> PB9_PWM
Routing:
- net PB9_PWM: track 0.00 -> 17.1 mm, vias 0 -> 2
- net /KicadJE_STM32F0/STM32F103C8/STM32_SDA1_PWM_PB9: track 14.5 -> 0.00 mm, vias 2 -> 0
- net PB2_R2: track 0.00 -> 13.0 mm
- net /KicadJE_STM32F0/STM32F103C8/STM32_boot1_PB2: track 13.0 -> 0.00 mm
- net Net-(D401-Pad2): track 0.00 -> 2.61 mm
- net /KicadJE_STM32F0/STM32F103C8/STM32_USB_P_PA12: track 38.4 -> 36.9 mm
- net GNDA: track 123.7 -> 124.8 mm
- net PWM_PA9: track 4.56 -> 3.78 mm
- net /KicadJE_STM32F0/STM32F103C8/STM32_SWDIO_PA13: track 14.3 -> 14.9 mm
