File: STM32F103C8.sch (KiCad schematic (older format))
At the start: 27 parts, among them J501 BOOT, J502 UART, J503 USB_B_Micro, U501 AMS1117-3.3, U502 STM32F103C8Tx, Y501 8 MHz

Commit message: Kicad 5.1
Parts:
- J503: symbol Connector:USB_B_Micro -> KicadJE_uP_DAC-rescue:USB_B_Micro-Connector
Changed lines of the file:
@@
 $EndComp
 $Comp
-L Envelope-cache-2018-08-04-13-00-04:GND #PWR?
+L KicadJE_uP_DAC-rescue:GND-Envelope-cache-2018-08-04-13-00-04 #PWR?
 U 1 1 5CEECDC2
 P 5375 4850
@@
 $EndComp
 $Comp
-L Envelope-cache-2018-08-04-13-00-04:GND #PWR?
+L KicadJE_uP_DAC-rescue:GND-Envelope-cache-2018-08-04-13-00-04 #PWR?
 U 1 1 5CEECDFC
 P 1875 2700
@@
 	7650 1350 7750 1350
 $Comp
-L Envelope-cache-2018-08-04-13-00-04:GND #PWR?
+L KicadJE_uP_DAC-rescue:GND-Envelope-cache-2018-08-04-13-00-04 #PWR?
 U 1 1 5CEECE25
 P 8200 1375
@@
 	1875 2700 1875 2650
 $Comp
-L Envelope-cache-2018-08-04-13-00-04:+5V #PWR?
+L KicadJE_uP_DAC-rescue:+5V-Envelope-cache-2018-08-04-13-00-04 #PWR?
 U 1 1 5CEECE43
 P 6275 2225
@@
 $EndComp
 $Comp
-L Envelope-cache-2018-08-04-13-00-04:GND #PWR?
+L KicadJE_uP_DAC-rescue:GND-Envelope-cache-2018-08-04-13-00-04 #PWR?
 U 1 1 5CEECE76
 P 7500 2575
@@
 $EndComp
 $Comp
-L Envelope-cache-2018-08-04-13-00-04:GND #PWR?
+L KicadJE_uP_DAC-rescue:GND-Envelope-cache-2018-08-04-13-00-04 #PWR?
 U 1 1 5CEF56B4
 P 3425 4950
@@
 SWDIO
 $Comp
-L Connector:USB_B_Micro J503
+L KicadJE_uP_DAC-rescue:USB_B_Micro-Connector J503
 U 1 1 5CF75CE4
 P 7975 4450
@@
 $EndComp
 $Comp
-L Envelope-cache-2018-08-04-13-00-04:+5V #PWR?
+L KicadJE_uP_DAC-rescue:+5V-Envelope-cache-2018-08-04-13-00-04 #PWR?
 U 1 1 5CF80739
 P 7475 3875
@@
 	7475 4175 7475 4250
 $Comp
-L Envelope-cache-2018-08-04-13-00-04:GND #PWR?
+L KicadJE_uP_DAC-rescue:GND-Envelope-cache-2018-08-04-13-00-04 #PWR?
 U 1 1 5CF835AC
 P 8025 4900
@@
 	7650 975  7750 975
 $Comp
-L Envelope-cache-2018-08-04-13-00-04:GND #PWR?
+L KicadJE_uP_DAC-rescue:GND-Envelope-cache-2018-08-04-13-00-04 #PWR?
 U 1 1 5D225372
 P 8200 1000
@@
 	8200 975  8200 1000
 $Comp
-L Envelope-cache-2018-08-04-13-00-04:+5V #PWR?
+L KicadJE_uP_DAC-rescue:+5V-Envelope-cache-2018-08-04-13-00-04 #PWR?
 U 1 1 5D22F628
 P 7200 950
