File: TH_555_VCO1.sch (KiCad schematic (older format))
At the start: 72 parts, among them J601 CV1, J602 FM_lin, J603 Sync, J604 PWM, J605 Ramp, J606 Tri, J608 555_Pulse, P601 Doepfer_Power_10pin, Q601 MMBT2222A, U601 TLC555, U602 TL074, U603 TL074

Commit message: Kicad 5.1
Parts:
- Q601: symbol MMBT2222A:MMBT2222A -> KicadJE_uP_DAC-rescue:MMBT2222A-MMBT2222A
Changed lines of the file:
@@
 $EndDescr
 $Comp
-L Envelope-cache-2018-08-04-13-00-04:+12V #PWR?
+L KicadJE_uP_DAC-rescue:+12V-Envelope-cache-2018-08-04-13-00-04 #PWR?
 U 1 1 5DD8FB32
 P 1675 1075
@@
 $EndComp
 $Comp
-L Envelope-cache-2018-08-04-13-00-04:GND #PWR?
+L KicadJE_uP_DAC-rescue:GND-Envelope-cache-2018-08-04-13-00-04 #PWR?
 U 1 1 5DD8FB4A
 P 1775 1275
@@
 $EndComp
 $Comp
-L Envelope-cache-2018-08-04-13-00-04:GND #PWR?
+L KicadJE_uP_DAC-rescue:GND-Envelope-cache-2018-08-04-13-00-04 #PWR?
 U 1 1 5DD8FB50
 P 775 1275
@@
 	2575 1100 2650 1100
 $Comp
-L Envelope-cache-2018-08-04-13-00-04:GND #PWR?
+L KicadJE_uP_DAC-rescue:GND-Envelope-cache-2018-08-04-13-00-04 #PWR?
 U 1 1 5DD8FB72
 P 2575 1100
@@
 $EndComp
 $Comp
-L Envelope-cache-2018-08-04-13-00-04:+12V #PWR?
+L KicadJE_uP_DAC-rescue:+12V-Envelope-cache-2018-08-04-13-00-04 #PWR?
 U 1 1 5DD8FB78
 P 2900 800
@@
 	4125 6475 4200 6475
 $Comp
-L Envelope-cache-2018-08-04-13-00-04:GND #PWR?
+L KicadJE_uP_DAC-rescue:GND-Envelope-cache-2018-08-04-13-00-04 #PWR?
 U 1 1 5DD8FBD4
 P 4900 6600
@@
 	1275 2625 1325 2625
 $Comp
-L Envelope-cache-2018-08-04-13-00-04:GND #PWR?
+L KicadJE_uP_DAC-rescue:GND-Envelope-cache-2018-08-04-13-00-04 #PWR?
 U 1 1 5DD9491F
 P 4050 1700
@@
 	5925 7125 5925 7350
 $Comp
-L Envelope-cache-2018-08-04-13-00-04:GND #PWR?
+L KicadJE_uP_DAC-rescue:GND-Envelope-cache-2018-08-04-13-00-04 #PWR?
 U 1 1 5DD9492C
 P 2400 3825
@@
 $EndComp
 $Comp
-L Envelope-cache-2018-08-04-13-00-04:GND #PWR?
+L KicadJE_uP_DAC-rescue:GND-Envelope-cache-2018-08-04-13-00-04 #PWR?
 U 1 1 5DD96A3E
 P 5925 7350
@@
 	4125 6900 4200 6900
 $Comp
-L Envelope-cache-2018-08-04-13-00-04:GND #PWR?
+L KicadJE_uP_DAC-rescue:GND-Envelope-cache-2018-08-04-13-00-04 #PWR?
 U 1 1 5DD97712
 P 4900 7025
@@
 	5925 4800 5925 4825
 $Comp
-L Envelope-cache-2018-08-04-13-00-04:GND #PWR?
+L KicadJE_uP_DAC-rescue:GND-Envelope-cache-2018-08-04-13-00-04 #PWR?
 U 1 1 5DDF056E
 P 5925 5125
@@
 	2300 4075 2200 4075
 $Comp
-L Envelope-cache-2018-08-04-13-00-04:GND #PWR?
+L KicadJE_uP_DAC-rescue:GND-Envelope-cache-2018-08-04-13-00-04 #PWR?
 U 1 1 5DE090D0
 P 2200 4375
@@
 $EndComp
 $Comp
-L Envelope-cache-2018-08-04-13-00-04:GND #PWR?
+L KicadJE_uP_DAC-rescue:GND-Envelope-cache-2018-08-04-13-00-04 #PWR?
 U 1 1 5DE473D9
 P 1950 3375
@@
 	2100 3075 2150 3075
 $Comp
-L Envelope-cache-2018-08-04-13-00-04:+12V #PWR?
+L KicadJE_uP_DAC-rescue:+12V-Envelope-cache-2018-08-04-13-00-04 #PWR?
 U 1 1 5DE56C72
 P 2400 3225
@@
 $EndComp
 $Comp
-L Envelope-cache-2018-08-04-13-00-04:+12V #PWR?
+L KicadJE_uP_DAC-rescue:+12V-Envelope-cache-2018-08-04-13-00-04 #PWR?
 U 1 1 5DE57234
 P 2200 3775
@@
 	5850 4700 6025 4700
 $Comp
-L MMBT2222A:MMBT2222A Q601
+L KicadJE_uP_DAC-rescue:MMBT2222A-MMBT2222A Q601
 U 1 1 5DE5C58C
 P 6550 4700
@@
 	5350 4300 5875 4300
 $Comp
-L Envelope-cache-2018-08-04-13-00-04:+12V #PWR?
+L KicadJE_uP_DAC-rescue:+12V-Envelope-cache-2018-08-04-13-00-04 #PWR?
 U 1 1 5DE7320A
 P 5875 4300
@@
 $EndComp
 $Comp
-L Envelope-cache-2018-08-04-13-00-04:+12V #PWR?
+L KicadJE_uP_DAC-rescue:+12V-Envelope-cache-2018-08-04-13-00-04 #PWR?
 U 1 1 5DED0DA1
 P 875 5825
@@
 	8625 5125 8800 5125
 $Comp
-L Envelope-cache-2018-08-04-13-00-04:+12V #PWR?
+L KicadJE_uP_DAC-rescue:+12V-Envelope-cache-2018-08-04-13-00-04 #PWR?
 U 1 1 5DFEB24C
 P 9350 5125
@@
 	5325 2900 5325 2625
 $Comp
-L Envelope-cache-2018-08-04-13-00-04:+12V #PWR?
+L KicadJE_uP_DAC-rescue:+12V-Envelope-cache-2018-08-04-13-00-04 #PWR?
 U 1 1 5E0786BD
 P 9175 750
@@
 	525  525  525  2100
 $Comp
-L Envelope-cache-2018-08-04-13-00-04:+12V #PWR?
+L KicadJE_uP_DAC-rescue:+12V-Envelope-cache-2018-08-04-13-00-04 #PWR?
 U 1 1 5DD8FB38
 P 850 1075
@@
 $EndComp
 $Comp
-L Envelope-cache-2018-08-04-13-00-04:GND #PWR?
+L KicadJE_uP_DAC-rescue:GND-Envelope-cache-2018-08-04-13-00-04 #PWR?
 U 1 1 5E3D265D
 P 1325 4175
